File: hw/doorbell.brd (EAGLE design)
At the start: 160 x 100 mm, 15 parts, among them IC1 LM2940

Commit message: updated schematic and board
Parts:
- removed C4: 22n, rcl:C025-024X044
- removed JP1: (no value), jumper:JP1
- removed R2: 10k, rcl:0207/10
- moved X2 14.5 mm to (78.7, 29.2), turned to 270 degrees
- moved R1 13.0 mm to (63.5, 35.6)
Connections:
- removed net N$129: JP1.2, R2.1, X2.2
- net GND: no longer C4.1
- net INPUT: now also U$1.A4, X2.2; no longer C4.2, JP1.1, R2.2, U$1.D2
Routing:
- net INPUT: track 45.7 -> 17.8 mm, vias 1 -> 0
- net +5V: track 68.9 -> 53.6 mm
- net N$129: track 12.7 -> 0.00 mm
- net GND: track 116.2 -> 113.6 mm, vias 2 -> 0
