File: hw/doorbell.sch (EAGLE design)
At the start: 15 parts, among them IC1 LM2940

Commit message: updated schematic and board
Parts:
- removed C4: 22n, rcl:C-EU025-024X044
- removed JP1: (no value), jumper:JP1E
- removed R2: 10k, rcl:R-EU_0207/10
Connections:
- removed net N$129: JP1.2, R2.1, X2-2.1
- net GND: no longer C4.1
- net INPUT: now also U$1.A4, X2-2.1; no longer C4.2, JP1.1, R2.2, U$1.D2
Changed lines of the file:
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@@
 <part name="R1" library="rcl" deviceset="R-EU_" device="0207/10" value="10k"/>
 <part name="P+1" library="supply1" deviceset="+5V" device=""/>
-<part name="R2" library="rcl" deviceset="R-EU_" device="0207/10" value="10k"/>
-<part name="JP1" library="jumper" deviceset="JP1E" device=""/>
-<part name="C4" library="rcl" deviceset="C-EU" device="025-024X044" value="22n"/>
-<part name="GND10" library="supply1" deviceset="GND" device=""/>
 <part name="R3" library="rcl" deviceset="R-EU_" device="0309/V"/>
 <part name="GND11" library="supply1" deviceset="GND" device=""/>
@@
 <instance part="R1" gate="G$1" x="71.12" y="106.68" rot="MR90"/>
 <instance part="P+1" gate="1" x="71.12" y="116.84" rot="MR0"/>
-<instance part="R2" gate="G$1" x="83.82" y="99.06" rot="MR0"/>
-<instance part="JP1" gate="A" x="83.82" y="109.22"/>
-<instance part="C4" gate="G$1" x="71.12" y="91.44" rot="R180"/>
-<instance part="GND10" gate="1" x="71.12" y="83.82" rot="MR0"/>
 <instance part="R3" gate="G$1" x="83.82" y="38.1"/>
 <instance part="GND11" gate="1" x="76.2" y="30.48"/>
@@
 </segment>
 <segment>
-<pinref part="C4" gate="G$1" pin="1"/>
-<pinref part="GND10" gate="1" pin="GND"/>
-<wire x1="71.12" y1="86.36" x2="71.12" y2="88.9" width="0.1524" layer="91"/>
-</segment>
-<segment>
 <wire x1="76.2" y1="33.02" x2="101.6" y2="33.02" width="0.1524" layer="91"/>
 <wire x1="101.6" y1="33.02" x2="101.6" y2="38.1" width="0.1524" layer="91"/>
@@
 </segment>
 </net>
-<net name="N$129" class="0">
-<segment>
-<pinref part="X2" gate="-2" pin="1"/>
-<pinref part="R2" gate="G$1" pin="1"/>
-<wire x1="96.52" y1="99.06" x2="93.98" y2="99.06" width="0.1524" layer="91"/>
-<pinref part="JP1" gate="A" pin="2"/>
-<wire x1="93.98" y1="99.06" x2="88.9" y2="99.06" width="0.1524" layer="91"/>
-<wire x1="86.36" y1="106.68" x2="93.98" y2="106.68" width="0.1524" layer="91"/>
-<wire x1="93.98" y1="106.68" x2="93.98" y2="99.06" width="0.1524" layer="91"/>
-<junction x="93.98" y="99.06"/>
-</segment>
-</net>
 <net name="INPUT" class="0">
-<segment>
-<pinref part="U$1" gate="G$1" pin="D2"/>
-<wire x1="17.78" y1="99.06" x2="15.24" y2="99.06" width="0.1524" layer="91"/>
-<label x="15.24" y="99.06" size="1.4224" layer="95" rot="R180" xref="yes"/>
-</segment>
 <segment>
 <pinref part="R1" gate="G$1" pin="1"/>
 <wire x1="71.12" y1="99.06" x2="71.12" y2="101.6" width="0.1524" layer="91"/>
-<pinref part="R2" gate="G$1" pin="2"/>
-<wire x1="78.74" y1="99.06" x2="76.2" y2="99.06" width="0.1524" layer="91"/>
+<pinref part="X2" gate="-2" pin="1"/>
+<wire x1="71.12" y1="99.06" x2="96.52" y2="99.06" width="0.1524" layer="91"/>
+<wire x1="71.12" y1="99.06" x2="71.12" y2="78.74" width="0.1524" layer="91"/>
 <junction x="71.12" y="99.06"/>
-<pinref part="JP1" gate="A" pin="1"/>
-<wire x1="76.2" y1="99.06" x2="71.12" y2="99.06" width="0.1524" layer="91"/>
-<wire x1="83.82" y1="106.68" x2="76.2" y2="106.68" width="0.1524" layer="91"/>
-<wire x1="76.2" y1="106.68" x2="76.2" y2="99.06" width="0.1524" layer="91"/>
-<junction x="76.2" y="99.06"/>
-<pinref part="C4" gate="G$1" pin="2"/>
-<wire x1="71.12" y1="96.52" x2="71.12" y2="99.06" width="0.1524" layer="91"/>
-<wire x1="71.12" y1="99.06" x2="60.96" y2="99.06" width="0.1524" layer="91"/>
-<label x="60.96" y="99.06" size="1.4224" layer="95" rot="R180" xref="yes"/>
-</segment>
-</net>
+<pinref part="U$1" gate="G$1" pin="A4"/>
+<wire x1="71.12" y1="78.74" x2="48.26" y2="78.74" width="0.1524" layer="91"/>
+</segment>
+</net>
